Commit message: saving both legs sensor vals

File: body.urdf (robot description, URDF)
Before this commit: robot robot, 3 links, 2 joints
Joints:
- joint Torso_bLeg: origin xyz=1 0 1 rpy=0 0 0 -> xyz=1 0 1.5 rpy=0 0 0
- joint Torso_fLeg: origin xyz=2 0 1 rpy=0 0 0 -> xyz=2 0 1.5 rpy=0 0 0

Commit message: random movement

File: body.urdf (robot description, URDF)
Before this commit: robot robot, 3 links, 2 joints
Joints:
- joint Torso_bLeg: origin xyz=1 0 1.5 rpy=0 0 0 -> xyz=1 0 1 rpy=0 0 0
- joint Torso_fLeg: origin xyz=2 0 1.5 rpy=0 0 0 -> xyz=2 0 1 rpy=0 0 0
